File: SirNano5V/SirNano5V.kicad_pcb (KiCad board)
At the start: 2 copper layers, 45.2 x 18 mm, 40 parts, among them J1 Conn_01x14, J2 Conn_01x14, J3 USB_B_Micro, U1 ATmega328PB-MU, U2 AP2210K-ADJ

Commit message: Dimensions Updated
Parts:
- moved J1 0.06 mm to (112.8, 62.8)
- moved J2 0.06 mm to (112.8, 47.6)
