File: SirNanoV2.0/SirNanoV2.0.sch (KiCad schematic (older format))
At the start: 35 parts, among them J1 Conn_01x14, J2 Conn_01x14, J3 USB_B_Micro, U1 ATmega328PB-MU, U2 AP7365-ADJ, U3 FT231XQ, Y1 20MHz

Commit message: Fuse Footprint changed
Parts:
- C10, C9: value 2.2uF -> 1uF
- F1: footprint Resistor_SMD:R_0805_2012Metric -> Resistor_SMD:R_1206_3216Metric
Changed lines of the file:
@@
 EESchema Schematic File Version 4
-LIBS:SirNanoV2-cache
+LIBS:SirNanoV2.0-cache
 EELAYER 29 0
 EELAYER END
@@
 F 0 "F1" H 10288 4096 50  0000 L CNN
 F 1 "500mA" H 10288 4005 50  0000 L CNN
-F 2 "Resistor_SMD:R_0805_2012Metric" H 10250 3850 50  0001 L CNN
+F 2 "Resistor_SMD:R_1206_3216Metric" H 10250 3850 50  0001 L CNN
 F 3 "~" H 10200 4050 50  0001 C CNN
 	1    10200 4050
@@
 P 4800 1250
 F 0 "C10" H 4682 1296 50  0000 R CNN
-F 1 "2.2uF" H 4682 1205 50  0000 R CNN
+F 1 "1uF" H 4682 1205 50  0000 R CNN
 F 2 "Capacitor_SMD:C_0805_2012Metric_Pad1.15x1.40mm_HandSolder" H 4838 1100 50  0001 C CNN
 F 3 "~" H 4800 1250 50  0001 C CNN
@@
 P 3500 1250
 F 0 "C9" H 3382 1296 50  0000 R CNN
-F 1 "2.2uF" H 3382 1205 50  0000 R CNN
+F 1 "1uF" H 3382 1205 50  0000 R CNN
 F 2 "Capacitor_SMD:C_0805_2012Metric_Pad1.15x1.40mm_HandSolder" H 3538 1100 50  0001 C CNN
 F 3 "~" H 3500 1250 50  0001 C CNN

Commit message: Part Numbers Added
Minor board Revisions
Parts:
- added C3: 100nF, Capacitor_SMD:C_0603_1608Metric, symbol Device:C
- C1, C11: Part (none) -> C42998
- C10, C9: footprint Capacitor_SMD:C_0805_2012Metric_Pad1.15x1.40mm_HandSolder -> Capacitor_SMD:C_0603_1608Metric_Pad1.05x0.95mm_HandSolder; Part (none) -> C29936
- C2, C4: Part (none) -> C105622
- C6: Part (none) -> C100042
- C7: Part (none) -> C29936
- C8: Part (none) -> C122643
- D1: Part (none) -> C12333
- F1: Part (none) -> C89657
- IO13: Part (none) -> C193191
- J3: Part (none) -> C132560
- L1: Part (none) -> C99366
- PWR1: Part (none) -> C118330
- R1, R2: Part (none) -> C325726
- R3: Part (none) -> C99198
- R5: Part (none) -> C304766
- R6: Part (none) -> C103426
- R7: Part (none) -> C163436
- RN1: Part (none) -> C164038
- RST1: Part (none) -> C231330
- RX1, TX1: Part (none) -> C205443
- U1: Part (none) -> 177-3693
- U2: Part (none) -> C264087
- U3: Part (none) -> 757-0045
- Y1: Part (none) -> C91586
Connections:
- net 3.3V: now also U3.11 (~RESET), C3.1
- net GND: now also C3.2
Changed lines of the file:
@@
 F 2 "Resistor_SMD:R_0603_1608Metric" V 9090 2840 50  0001 C CNN
 F 3 "~" H 9050 2850 50  0001 C CNN
+F 4 "C99198" H 9050 2850 50  0001 C CNN "Part"
 	1    9050 2850
 	-1   0    0    -1
@@
 F 2 "LED_SMD:LED_0603_1608Metric" H 7300 2150 50  0001 C CNN
 F 3 "~" H 7300 2150 50  0001 C CNN
+F 4 "C205443" H 7300 2150 50  0001 C CNN "Part"
 	1    7300 2150
 	1    0    0    -1
@@
 F 2 "Button_Switch_SMD:SW_SPST_B3U-1000P-B" H 8700 3300 50  0001 C CNN
 F 3 "~" H 8700 3300 50  0001 C CNN
+F 4 "C231330" H 8700 3100 50  0001 C CNN "Part"
 	1    8700 3100
 	-1   0    0    -1
@@
 F 2 "Inductor_SMD:L_0805_2012Metric_Pad1.15x1.40mm_HandSolder" H 4500 2350 50  0001 C CNN
 F 3 "~" H 4500 2350 50  0001 C CNN
+F 4 "C99366" V 4500 2350 50  0001 C CNN "Part"
 	1    4500 2350
 	0    1    -1   0
@@
 F 2 "Resistor_SMD:R_0603_1608Metric" V 9740 4590 50  0001 C CNN
 F 3 "~" H 9700 4600 50  0001 C CNN
+F 4 "C325726" V 9700 4600 50  0001 C CNN "Part"
 	1    9700 4600
 	0    1    -1   0
@@
 F 2 "Resistor_SMD:R_0603_1608Metric" V 9740 4790 50  0001 C CNN
 F 3 "~" H 9700 4800 50  0001 C CNN
+F 4 "C325726" V 9700 4800 50  0001 C CNN "Part"
 	1    9700 4800
 	0    1    -1   0
@@
 F 2 "Capacitor_SMD:C_0603_1608Metric_Pad1.05x0.95mm_HandSolder" H 4838 2400 50  0001 C CNN
 F 3 "~" H 4800 2550 50  0001 C CNN
+F 4 "C29936" H 4800 2550 50  0001 C CNN "Part"
 	1    4800 2550
 	-1   0    0    -1
@@
 F 2 "LED_SMD:LED_0603_1608Metric" H 7300 2550 50  0001 C CNN
 F 3 "~" H 7300 2550 50  0001 C CNN
+F 4 "C205443" H 7300 2550 50  0001 C CNN "Part"
 	1    7300 2550
 	1    0    0    -1
@@
 F 2 "LED_SMD:LED_0603_1608Metric" H 7300 2950 50  0001 C CNN
 F 3 "~" H 7300 2950 50  0001 C CNN
+F 4 "C118330" H 7300 2950 50  0001 C CNN "Part"
 	1    7300 2950
 	-1   0    0    -1
@@
 F 2 "LED_SMD:LED_0603_1608Metric" H 7300 3300 50  0001 C CNN
 F 3 "~" H 7300 3300 50  0001 C CNN
+F 4 "C193191" H 7300 3300 50  0001 C CNN "Part"
 	1    7300 3300
 	-1   0    0    -1
@@
 F 2 "Resistor_SMD:R_1206_3216Metric" H 10250 3850 50  0001 L CNN
 F 3 "~" H 10200 4050 50  0001 C CNN
+F 4 "C89657" H 10200 4050 50  0001 C CNN "Part"
 	1    10200 4050
 	-1   0    0    -1
@@
 F 2 "Capacitor_Tantalum_SMD:CP_EIA-3216-12_Kemet-S" H 10038 5000 50  0001 C CNN
 F 3 "~" H 10000 5150 50  0001 C CNN
+F 4 "C122643" H 10000 5150 50  0001 C CNN "Part"
 	1    10000 5150
 	1    0    0    -1
@@
 F 2 "Capacitor_SMD:C_0603_1608Metric" H 3188 3200 50  0001 C CNN
 F 3 "~" H 3150 3350 50  0001 C CNN
+F 4 "C42998" H 3150 3350 50  0001 C CNN "Part"
 	1    3150 3350
 	-1   0    0    -1
@@
 F 2 "Package_DFN_QFN:QFN-32-1EP_5x5mm_P0.5mm_EP3.1x3.1mm" H 4050 4300 50  0001 C CIN
 F 3 "http://ww1.microchip.com/downloads/en/DeviceDoc/40001906C.pdf" H 4050 4300 50  0001 C CNN
+F 4 "177-3693" H 4050 4300 50  0001 C CNN "Part"
 	1    4050 4300
 	1    0    0    -1
@@
 F 2 "Package_DFN_QFN:QFN-20-1EP_4x4mm_P0.5mm_EP2.5x2.5mm" H 8400 4100 50  0001 C CNN
 F 3 "http://www.ftdichip.com/Products/ICs/FT231X.html" H 7900 4950 50  0001 C CNN
+F 4 "757-0045" H 7900 4950 50  0001 C CNN "Part"
 	1    7900 4950
 	-1   0    0    -1
@@
 F 2 "Capacitor_SMD:C_0603_1608Metric" H 9088 5000 50  0001 C CNN
 F 3 "~" H 9050 5150 50  0001 C CNN
+F 4 "C105622" H 9050 5150 50  0001 C CNN "Part"
 	1    9050 5150
 	-1   0    0    -1
@@
 F 2 "Connector_USB:USB_Micro-B_Molex_47346-0001" H 10800 4600 50  0001 C CNN
 F 3 "~" H 10800 4600 50  0001 C CNN
+F 4 "C132560" H 10650 4650 50  0001 C CNN "Part"
 	1    10650 4650
 	-1   0    0    -1
@@
 F 2 "Capacitor_SMD:C_0603_1608Metric" H 10238 5000 50  0001 C CNN
 F 3 "~" H 10200 5150 50  0001 C CNN
+F 4 "C100042" H 10200 5150 50  0001 C CNN "Part"
 	1    10200 5150
 	1    0    0    -1
@@
 Connection ~ 8550 6050
 Wire Wire Line
-	8550 6050 9050 6050
-$Comp
-L Device:C C11
-U 1 1 5DA62F39
-P 6850 4750
-F 0 "C11" H 6965 4796 50  0000 L CNN
-F 1 "100nF" H 6965 4705 50  0000 L CNN
-F 2 "Capacitor_SMD:C_0603_1608Metric" H 6888 4600 50  0001 C CNN
-F 3 "~" H 6850 4750 50  0001 C CNN
-	1    6850 4750
-	0    -1   1    0
-$EndComp
+	8550 6050 8650 6050
 Wire Wire Line
 	7200 4750 7000 4750
@@
 Wire Wire Line
 	6000 2900 6350 2900
-$Comp
-L Device:CP C10
-U 1 1 5DB9B9CE
-P 4800 1250
-F 0 "C10" H 4682 1296 50  0000 R CNN
-F 1 "1uF" H 4682 1205 50  0000 R CNN
-F 2 "Capacitor_SMD:C_0805_2012Metric_Pad1.15x1.40mm_HandSolder" H 4838 1100 50  0001 C CNN
-F 3 "~" H 4800 1250 50  0001 C CNN
-	1    4800 1250
-	-1   0    0    -1
-$EndComp
-$Comp
-L Device:CP C9
-U 1 1 5DB9B9D5
-P 3500 1250
-F 0 "C9" H 3382 1296 50  0000 R CNN
-F 1 "1uF" H 3382 1205 50  0000 R CNN
-F 2 "Capacitor_SMD:C_0805_2012Metric_Pad1.15x1.40mm_HandSolder" H 3538 1100 50  0001 C CNN
-F 3 "~" H 3500 1250 50  0001 C CNN
-	1    3500 1250
-	-1   0    0    -1
-$EndComp
 Wire Wire Line
 	4800 1100 4800 900
@@
 Wire Wire Line
 	3500 900  3500 1100
-Wire Wire Line
-	4050 1200 4050 1300
-Connection ~ 4050 1300
 Wire Wire Line
 	4050 1300 4050 1550
@@
 F 2 "Crystal:Resonator_SMD_muRata_CSTxExxV-3Pin_3.0x1.1mm" H 5425 3750 50  0001 C CNN
 F 3 "~" H 5425 3750 50  0001 C CNN
+F 4 "C91586" V 5450 3750 50  0001 C CNN "Part"
 	1    5450 3750
 	0    -1   -1   0
@@
 F 2 "Capacitor_SMD:C_0603_1608Metric" H 9388 5000 50  0001 C CNN
 F 3 "~" H 9350 5150 50  0001 C CNN
+F 4 "C105622" H 9350 5150 50  0001 C CNN "Part"
 	1    9350 5150
 	1    0    0    -1
@@
 Wire Wire Line
 	8850 850  8700 850
-$Comp
-L Power_Protection:PRTR5V0U2X D1
-U 1 1 5DA68898
-P 6000 1400
-F 0 "D1" H 6543 1445 50  0000 L CNN
-F 1 "PRTR5V0U2X" H 6543 1355 50  0000 L CNN
-F 2 "Package_TO_SOT_SMD:SOT-143" H 6060 1400 50  0001 C CNN
-F 3 "https://assets.nexperia.com/documents/data-sheet/PRTR5V0U2X.pdf" H 6060 1400 50  0001 C CNN
-	1    6000 1400
-	1    0    0    -1
-$EndComp
 Text GLabel 5400 1400 0    50   Input ~ 0
 D+
@@
 F 2 "Package_TO_SOT_SMD:SOT-23-5" H 4050 1325 50  0001 C CNN
 F 3 "https://www.diodes.com/assets/Datasheets/AP2204.pdf" H 4050 1100 50  0001 C CNN
+F 4 "C264087" H 4050 1000 50  0001 C CNN "Part"
 	1    4050 1000
 	1    0    0    -1
@@
 F 2 "Resistor_SMD:R_0603_1608Metric" V 1340 2190 50  0001 C CNN
 F 3 "~" H 1300 2200 50  0001 C CNN
+F 4 "C304766" V 1300 2200 50  0001 C CNN "Part"
 	1    1300 2200
 	0    1    -1   0
@@
 F 2 "Resistor_SMD:R_0603_1608Metric" V 1340 2890 50  0001 C CNN
 F 3 "~" H 1300 2900 50  0001 C CNN
+F 4 "C103426" V 1300 2900 50  0001 C CNN "Part"
 	1    1300 2900
 	0    1    -1   0
@@
 F 2 "Resistor_SMD:R_0603_1608Metric" V 2290 2540 50  0001 C CNN
 F 3 "~" H 2250 2550 50  0001 C CNN
+F 4 "C163436" V 2250 2550 50  0001 C CNN "Part"
 	1    2250 2550
 	0    1    -1   0
@@
 F 2 "Resistor_SMD:R_Array_Concave_4x0603" V 6825 2800 50  0001 C CNN
 F 3 "~" H 6550 2800 50  0001 C CNN
+F 4 "C164038" V 6550 2800 50  0001 C CNN "Part"
 	1    6550 2800
 	0    1    1    0
@@
 	1700 2900 1600 2900
 Connection ~ 1600 2900
+Wire Wire Line
+	8650 5325 8650 4950
+Wire Wire Line
+	8650 4950 8600 4950
+Wire Wire Line
+	8650 5625 8650 6050
+Connection ~ 8650 6050
+Wire Wire Line
+	8650 6050 9050 6050
+Wire Wire Line
+	8650 4950 8650 4350
+Connection ~ 8650 4950
+$Comp
+L Device:C C3
+U 1 1 5E251200
+P 8650 5475
+F 0 "C3" H 8765 5521 50  0000 L CNN
+F 1 "100nF" H 8765 5430 50  0000 L CNN
+F 2 "Capacitor_SMD:C_0603_1608Metric" H 8688 5325 50  0001 C CNN
+F 3 "~" H 8650 5475 50  0001 C CNN
+F 4 "C42998" H 8650 5475 50  0001 C CNN "Part"
+	1    8650 5475
+	1    0    0    -1
+$EndComp
+$Comp
+L Device:CP C10
+U 1 1 5E27965A
+P 4800 1250
+F 0 "C10" H 4682 1296 50  0000 R CNN
+F 1 "1uF" H 4682 1205 50  0000 R CNN
+F 2 "Capacitor_SMD:C_0603_1608Metric_Pad1.05x0.95mm_HandSolder" H 4838 1100 50  0001 C CNN
+F 3 "~" H 4800 1250 50  0001 C CNN
+F 4 "C29936" H 4800 1250 50  0001 C CNN "Part"
+	1    4800 1250
+	-1   0    0    -1
+$EndComp
+$Comp
+L Device:CP C9
+U 1 1 5E288501
+P 3500 1250
+F 0 "C9" H 3382 1296 50  0000 R CNN
+F 1 "1uF" H 3382 1205 50  0000 R CNN
+F 2 "Capacitor_SMD:C_0603_1608Metric_Pad1.05x0.95mm_HandSolder" H 3538 1100 50  0001 C CNN
+F 3 "~" H 3500 1250 50  0001 C CNN
+F 4 "C29936" H 3500 1250 50  0001 C CNN "Part"
+	1    3500 1250
+	-1   0    0    -1
+$EndComp
+$Comp
+L Power_Protection:PRTR5V0U2X D1
+U 1 1 5DA68898
+P 6000 1400
+F 0 "D1" H 6350 1200 50  0000 L CNN
+F 1 "PRTR5V0U2X" H 6350 1125 50  0000 L CNN
+F 2 "Package_TO_SOT_SMD:SOT-143" H 6060 1400 50  0001 C CNN
+F 3 "https://assets.nexperia.com/documents/data-sheet/PRTR5V0U2X.pdf" H 6060 1400 50  0001 C CNN
+F 4 "C12333" H 6000 1400 50  0001 C CNN "Part"
+	1    6000 1400
+	1    0    0    -1
+$EndComp
+$Comp
+L Device:C C11
+U 1 1 5E2607AF
+P 6850 4750
+F 0 "C11" V 6975 4800 50  0000 L CNN
+F 1 "100nF" V 6975 4500 50  0000 L CNN
+F 2 "Capacitor_SMD:C_0603_1608Metric" H 6888 4600 50  0001 C CNN
+F 3 "~" H 6850 4750 50  0001 C CNN
+F 4 "C42998" H 6850 4750 50  0001 C CNN "Part"
+	1    6850 4750
+	0    -1   -1   0
+$EndComp
 $EndSCHEMATC

Commit message: SirNano5V, SirNano3V3, SirNano1V8 removed
Parts:
- removed C7: 1uF, Capacitor_SMD:C_0603_1608Metric_Pad1.05x0.95mm_HandSolder, symbol Device:CP
- added C?: 100nF, Capacitor_SMD:C_0603_1608Metric, symbol Device:C
Connections:
- net GND: now also C?.2
- net VCC: now also C?.1
Changed lines of the file:
@@
-$EndComp
-$Comp
-L Device:CP C7
-U 1 1 5D3FC5C3
-P 4800 2550
-F 0 "C7" H 4682 2596 50  0000 R CNN
-F 1 "1uF" H 4682 2505 50  0000 R CNN
-F 2 "Capacitor_SMD:C_0603_1608Metric_Pad1.05x0.95mm_HandSolder" H 4838 2400 50  0001 C CNN
-F 3 "~" H 4800 2550 50  0001 C CNN
-F 4 "C29936" H 4800 2550 50  0001 C CNN "Part"
-	1    4800 2550
-	-1   0    0    -1
 $EndComp
 $Comp
@@
 	0    -1   -1   0
 $EndComp
+$Comp
+L Device:C C?
+U 1 1 5DF28D4F
+P 4800 2550
+F 0 "C?" H 4915 2596 50  0000 L CNN
+F 1 "100nF" H 4915 2505 50  0000 L CNN
+F 2 "Capacitor_SMD:C_0603_1608Metric" H 4838 2400 50  0001 C CNN
+F 3 "~" H 4800 2550 50  0001 C CNN
+F 4 "C42998" H 4800 2550 50  0001 C CNN "Part"
+	1    4800 2550
+	-1   0    0    -1
+$EndComp
 $EndSCHEMATC
